File: Carte de puissance.kicad_sch (KiCad schematic)
At the start: 96 parts, among them J1 5v external regulator, J2 other external regulator, J3 Pi_pwr, J4 Pi_data, J5 BAU1, J6 BAU2, J7 BAU3, J8 BAU4, J9 Programming, Q1 GSFP6901, Q2 GSFP6901, Q3 BC847, Q4 BC847, Q6 BC847, Q7 GSFP6901, Q8 BC847, SW1 SW_Push, SW2 Emergency switch (NC), U1 WeAct TPS5450 buck stepdown (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, U10 DPC817-B, U11 DPC817-B, U12 DPC817-B, U13 ATtiny1626-X, U2 WeAct TPS5450 buck stepdown (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, U3 WeAct TPS5450 buck stepdown (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, U5 PAC1811, U6 H11L1, U7 DPC817-B, U8 DPC817-B, U9 DPC817-B

Commit message: Carte principale fini
Parts:
- added J10: Pi external regulator, MR30PB:MR30PB, symbol Connector:Conn_01x03_Socket
- added J11: External enable, Connector_PinHeader_2.54mm:PinHeader_1x01_P2.54mm_Vertical, symbol Connector:Conn_01x01_Pin
- renumbered ALM4 to ALM1, ALM3 to ALM2, ALM2 to ALM3, ALM1 to ALM4, C11 to C1, C9 to C10, C5 to C11, C7 to C12, C6 to C13, C10 to C14, C4 to C15, C15 to C2, C13 to C3, C14 to C4, C8 to C5, C3 to C6, C1 to C7, C2 to C8, C12 to C9, D3 to D1, D5 to D2, D1 to D3, D7 to D5, D2 to D6, D6 to D7, F4 to F0, F5 to F1, F3 to F2, F2 to F3, F1 to F4, H4 to H3, H3 to H4, J9 to J1, J4 to J2, J1 to J3, J2 to J4, J8 to J5, J7 to J6, J6 to J7, J5 to J8, J3 to J9, Q3 to Q1, Q1 to Q3, Q7 to Q4, Q4 to Q5, Q8 to Q7, R22 to R1, R24 to R10, R6 to R11, R7 to R12, R25 to R13, R10 to R14, R26 to R15, R9 to R16, R23 to R17, R8 to R18, R16 to R19, R3 to R2, R15 to R20, R13 to R21, R12 to R22, R20 to R23, R19 to R24, R18 to R25, R17 to R26, R4 to R3, R21 to R4, R1 to R5, R2 to R6, R5 to R7, R14 to R8, R11 to R9, U5 to U1, U11 to U10, U10 to U11, U9 to U12, U13 to U2, U1 to U3, U2 to U4, U3 to U5, U8 to U6, U6 to U8, U12 to U9
Connections:
- net +VSW: now also J10.3 (Pin_3)
- net +V_PI: now also J10.1 (Pin_1)
- net GND: now also J10.2 (Pin_2)
- net at Q5.3 (C), U3.3 (EN): now also J11.1 (Pin_1)
